Commit message: 基础仿真和小车手柄控制\视觉已添加

File: scout_description/urdf/scout_v2.gazebo.xacro (robot description, xacro)
@@ -78,3 +78,188 @@
         </plugin>
     </gazebo>
+    <!-- ========== Intel RealSense D435 (front), pal-robotics plugin ==========
+         Uses realsense_gazebo_plugin (vendored in this workspace): four
+         independent Gazebo sensors on one link (depth / color / infra1 /
+         infra2) aggregated by librealsense_gazebo_plugin.so, publishing the
+         realsense-ros topic tree (/camera/color/image_raw, .../aligned_depth_
+         to_color/image_raw, infra1/2, point cloud with correct PCL rgb
+         packing; out-of-range points are NaN, not inf).
+         D435 parameters: depth 87 deg H-FOV @ 848x480 (yields the spec 58 deg
+         V-FOV), color 69 deg H-FOV, depth range 0.3-10 m, rgb far clip 200 m.
+         The infra cameras run at 1 Hz on purpose: nothing in this sim
+         consumes them (stereo depth is not simulated), and every camera is
+         an extra render pass.
+         Sensor names must be <prefix> + depth/color/ired1/ired2 (hardcoded
+         lookup in RealSensePlugin::Load). -->
+    <link name="camera_link">
+        <visual>
+            <origin xyz="0 0 0" rpy="0 0 0"/>
+            <geometry>
+                <!-- D435 body: 90 x 25 x 25 mm, width along Y -->
+                <box size="0.025 0.09 0.025"/>
+            </geometry>
+            <material name="d435_dark">
+                <color rgba="0.15 0.15 0.15 1"/>
+            </material>
+        </visual>
+    </link>
+    <joint name="camera_joint" type="fixed">
+        <parent link="base_link"/>
+        <child link="camera_link"/>
+        <!-- front panel, ~0.33 m above ground -->
+        <origin xyz="0.44 0 0.10" rpy="0 0 0"/>
+    </joint>
+    <!-- Optical frames (data convention: z forward, x right, y down).
+         The plugin stamps messages with these names; robot_state_publisher
+         provides the transforms. -->
+    <link name="camera_color_optical_frame"/>
+    <joint name="camera_color_optical_joint" type="fixed">
+        <parent link="camera_link"/>
+        <child link="camera_color_optical_frame"/>
+        <origin xyz="0 0 0" rpy="-1.5708 0 -1.5708"/>
+    </joint>
+    <link name="camera_depth_optical_frame"/>
+    <joint name="camera_depth_optical_joint" type="fixed">
+        <parent link="camera_link"/>
+        <child link="camera_depth_optical_frame"/>
+        <origin xyz="0 0 0" rpy="-1.5708 0 -1.5708"/>
+    </joint>
+    <link name="camera_infra1_optical_frame"/>
+    <joint name="camera_infra1_optical_joint" type="fixed">
+        <parent link="camera_link"/>
+        <child link="camera_infra1_optical_frame"/>
+        <origin xyz="0 0 0" rpy="-1.5708 0 -1.5708"/>
+    </joint>
+    <link name="camera_infra2_optical_frame"/>
+    <joint name="camera_infra2_optical_joint" type="fixed">
+        <parent link="camera_link"/>
+        <child link="camera_infra2_optical_frame"/>
+        <origin xyz="0 0 0" rpy="-1.5708 0 -1.5708"/>
+    </joint>
+    <!-- depth module: 87 deg FOV, 848x480, 0.3-10 m -->
+    <gazebo reference="camera_link">
+        <sensor name="cameradepth" type="depth">
+            <update_rate>30</update_rate>
+            <always_on>true</always_on>
+            <visualize>false</visualize>
+            <camera name="depth">
+                <horizontal_fov>1.51844</horizontal_fov>
+                <image>
+                    <width>848</width>
+                    <height>480</height>
+                </image>
+                <clip>
+                    <near>0.3</near>
+                    <far>10.0</far>
+                </clip>
+                <noise>
+                    <type>gaussian</type>
+                    <mean>0.0</mean>
+                    <stddev>0.01</stddev>
+                </noise>
+            </camera>
+        </sensor>
+    </gazebo>
+    <!-- rgb camera: 69 deg FOV, far clip 200 m so the image is not truncated -->
+    <gazebo reference="camera_link">
+        <sensor name="cameracolor" type="camera">
+            <update_rate>30</update_rate>
+            <always_on>true</always_on>
+            <visualize>false</visualize>
+            <camera name="color">
+                <horizontal_fov>1.2042</horizontal_fov>
+                <image>
+                    <width>848</width>
+                    <height>480</height>
+                    <!-- plugin only supports RGB_INT8 / L_INT8 -->
+                    <format>RGB_INT8</format>
+                </image>
+                <clip>
+                    <near>0.1</near>
+                    <far>200.0</far>
+                </clip>
+                <noise>
+                    <type>gaussian</type>
+                    <mean>0.0</mean>
+                    <stddev>0.007</stddev>
+                </noise>
+            </camera>
+        </sensor>
+    </gazebo>
+    <!-- infrared stereo pair, 1 Hz (unused in sim, saves render passes) -->
+    <gazebo reference="camera_link">
+        <sensor name="cameraired1" type="camera">
+            <update_rate>1</update_rate>
+            <always_on>true</always_on>
+            <visualize>false</visualize>
+            <camera name="ired1">
+                <horizontal_fov>1.51844</horizontal_fov>
+                <image>
+                    <width>848</width>
+                    <height>480</height>
+                    <format>L_INT8</format>
+                </image>
+                <clip>
+                    <near>0.3</near>
+                    <far>10.0</far>
+                </clip>
+                <noise>
+                    <type>gaussian</type>
+                    <mean>0.0</mean>
+                    <stddev>0.05</stddev>
+                </noise>
+            </camera>
+        </sensor>
+    </gazebo>
+    <gazebo reference="camera_link">
+        <sensor name="cameraired2" type="camera">
+            <update_rate>1</update_rate>
+            <always_on>true</always_on>
+            <visualize>false</visualize>
+            <camera name="ired2">
+                <horizontal_fov>1.51844</horizontal_fov>
+                <image>
+                    <width>848</width>
+                    <height>480</height>
+                    <format>L_INT8</format>
+                </image>
+                <clip>
+                    <near>0.3</near>
+                    <far>10.0</far>
+                </clip>
+                <noise>
+                    <type>gaussian</type>
+                    <mean>0.0</mean>
+                    <stddev>0.05</stddev>
+                </noise>
+            </camera>
+        </sensor>
+    </gazebo>
+    <!-- model-level aggregator plugin: publishes the realsense-ros topic tree -->
+    <gazebo>
+        <plugin name="d435" filename="librealsense_gazebo_plugin.so">
+            <prefix>camera</prefix>
+            <depthUpdateRate>30.0</depthUpdateRate>
+            <colorUpdateRate>30.0</colorUpdateRate>
+            <infraredUpdateRate>1.0</infraredUpdateRate>
+            <depthTopicName>aligned_depth_to_color/image_raw</depthTopicName>
+            <depthCameraInfoTopicName>depth/camera_info</depthCameraInfoTopicName>
+            <colorTopicName>color/image_raw</colorTopicName>
+            <colorCameraInfoTopicName>color/camera_info</colorCameraInfoTopicName>
+            <infrared1TopicName>infra1/image_raw</infrared1TopicName>
+            <infrared1CameraInfoTopicName>infra1/camera_info</infrared1CameraInfoTopicName>
+            <infrared2TopicName>infra2/image_raw</infrared2TopicName>
+            <infrared2CameraInfoTopicName>infra2/camera_info</infrared2CameraInfoTopicName>
+            <colorOpticalframeName>camera_color_optical_frame</colorOpticalframeName>
+            <depthOpticalframeName>camera_depth_optical_frame</depthOpticalframeName>
+            <infrared1OpticalframeName>camera_infra1_optical_frame</infrared1OpticalframeName>
+            <infrared2OpticalframeName>camera_infra2_optical_frame</infrared2OpticalframeName>
+            <rangeMinDepth>0.3</rangeMinDepth>
+            <rangeMaxDepth>10.0</rangeMaxDepth>
+            <pointCloud>true</pointCloud>
+            <pointCloudTopicName>depth/color/points</pointCloudTopicName>
+            <pointCloudCutoff>0.3</pointCloudCutoff>
+            <pointCloudCutoffMax>10.0</pointCloudCutoffMax>
+        </plugin>
+    </gazebo>
 </robot>
